File: Plantilla.kicad_sch (KiCad schematic)
At the start: 12 parts, among them J1 Screw_Terminal_01x03, Q1 IRF540N, U1 TIMER 555

Commit message: Se ha redibujado la capa de relleno de cobre.
Other:
- note added: "DIMMER 5"
- note removed: "DIMMER 555"
Changed lines of the file:
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@@
 		(company "UPNA")
 	)
-	(text "DIMMER 555"
+	(text "DIMMER 5"
 		(exclude_from_sim no)
 		(at 151.13 45.212 0)

Commit message: Añade identificación al esquemático
Other:
- note added: "Izan - sesión 1"
Changed lines of the file:
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@@
+		)
+	)
+	(text "Izan - sesión 1"
+		(exclude_from_sim no)
+		(at 87.884 146.304 0)
+		(effects
+			(font
+				(size 1.27 1.27)
+			)
 		)
 	)
@@
 			(justify left bottom)
 		)
-		(property "Clase de red" "GND"
+		(property "Netclass" "GND"
 			(at 168.3385 140.97 0)
 			(show_name no)
@@
 			(justify left bottom)
 		)
-		(property "Clase de red" "VCC"
+		(property "Netclass" "VCC"
 			(at 141.6685 91.44 0)
 			(show_name no)
@@
 			(justify right bottom)
 		)
-		(property "Clase de red" "SIGNAL"
+		(property "Netclass" "SIGNAL"
 			(at 181.0385 128.27 0)
 			(show_name no)
