File: Plantilla.kicad_pcb (KiCad board)
At the start: 2 copper layers, 60 x 30.1 mm, 12 parts, among them J1 Screw_Terminal_01x03, Q1 IRF540N, U1 TIMER 555

Commit message: Añade identificación en serigrafía PCB
Other:
- board text added: "Izan - sesión 1"
Changed lines of the file:
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@@
 		(layer "Edge.Cuts")
+	)
+	(gr_text "Izan - sesión 1"
+		(at 136.5 92 0)
+		(layer "F.SilkS")
+		(effects
+			(font
+				(size 1 1)
+				(thickness 0.1)
+			)
+			(justify left bottom)
+		)
 	)
 	(segment
