File: Plantilla.kicad_pcb (KiCad board)
At the start: 2 copper layers, 60 x 30.1 mm, 12 parts, among them J1 Screw_Terminal_01x03, Q1 IRF540N, U1 TIMER 555

Commit message: Nuevo LED en paralelo
Parts:
- added D4: LED, Diode_SMD:D_1206_3216Metric, F.Cu at (156.0, 102.1)
Routing:
- net Net-(D3-A): track 1.97 -> 7.66 mm
